File: PowerModule_PTH_Terminal3.5mm.kicad_pcb (KiCad board)
At the start: 2 copper layers, 26.3 x 20 mm, 5 parts, among them J1 Conn_01x05, J2 Conn_01x05, J3 Screw_Terminal

Commit message: Fix the wrong side connectors
Parts:
- moved J3 0.20 mm to (144.4, 101.6)
Connections:
- J1 pad 1: VDC -> GND
- J1 pad 2: VDC -> GND
- J1 pad 4: GND -> VDC
- J1 pad 5: GND -> VDC
- J2 pad 1: GND -> VDC
- J2 pad 2: GND -> VDC
- J2 pad 4: VDC -> GND
- J2 pad 5: VDC -> GND
Routing:
- net GND: track 41.8 -> 0.00 mm, vias 44 -> 55
- net VDC: vias 0 -> 15
- added copper zone on B.Cu, net VDC
Other:
- board text added: "PnP Power Module 3.5mm Screw Terminal"
- board text removed: "PnP Power Module Screw Terminal"
